File: KiCad/Non-split-keebs.kicad_sch (KiCad schematic)
At the start: 194 parts, among them J1 USB_C_Receptacle_USB2.0_16P, U1 ESP32-S3-WROOM-1, U2 AMS1117-3.3

Commit message: pcb files changes
Parts:
- removed H2, H4, H6, H8: MountingHole, MountingHole:MountingHole_3.2mm_M3, symbol Mechanical:MountingHole
Connections:
- net +5V: now also C11.1, J1.A4 (VBUS), J1.A9 (VBUS), J1.B4 (VBUS), J1.B9 (VBUS), U2.3 (VI)
