File: KiCad/Non-split-keebs.kicad_pcb (KiCad board)
At the start: 2 copper layers, 368.4 x 157.2 mm, 194 parts, among them J1 USB_C_Receptacle_USB2.0_16P, U1 ESP32-S3-WROOM-1, U2 AMS1117-3.3

Commit message: pcb files changes
Parts:
- removed H2, H4, H6, H8: MountingHole, MountingHole:MountingHole_3.2mm_M3
- D1, D10, D11, D12, D13, D14, D15, D16, D17, D18, D19, D2, D20, D21, D22, D23, D24, D25, D26, D27, D28, D29, D3, D30, D31, D32, D33, D34, D35, D36, D37, D38, D39, D4, D40, D41, D42, D43, D44, D45, D46, D47, D48, D49, D5, D50, D51, D52, D53, D54, D55, D56, D57, D58, D59, D6, D60, D61, D62, D63, D64, D65, D66, D67, D68, D69, D7, D70, D71, D72, D73, D74, D75, D76, D77, D78, D79, D8, D80, D81, D82, D83, D84, D85, D86, D87, D88, D9: moved to F.Cu
- moved H1 336.5 mm to (291.4, 259.4)
- moved H7 272.3 mm to (291.4, 283.3)
- moved H3 247.9 mm to (291.4, 267.4)
- moved H5 175.1 mm to (291.4, 275.3)
- moved C12 32.8 mm to (212.1, 22.5)
- moved U2 31.1 mm to (217.6, 17.8), turned to 0 degrees
- moved C11 17.8 mm to (209.9, 22.6)
- moved R4 14.0 mm to (161.2, 15.8)
- moved C2 13.8 mm to (157.7, 15.9)
- moved U1 13.7 mm to (172.7, 18.4)
- moved C1 10.3 mm to (157.7, 13.3)
- moved J1 6.91 mm to (207.4, 15.2)
- moved R2 6.61 mm to (205.3, 21.7)
- moved R1 6.33 mm to (208.0, 21.7)
- moved D12 1.44 mm to (281.8, 51.1), turned to 180 degrees
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Connections:
- net Net-(U2-VI) renamed +5V
Routing:
- net ROW1: track 470.0 -> 552.2 mm, vias 5 -> 34
- net ROW2: track 478.1 -> 434.8 mm, vias 7 -> 29
- net COL9: track 214.5 -> 176.3 mm
- net COL11: track 269.9 -> 232.9 mm, vias 1 -> 2
- net COL12: track 288.4 -> 251.5 mm, vias 1 -> 2
- net COL10: track 252.0 -> 215.6 mm, vias 1 -> 2
- net +3V3: track 52.0 -> 83.3 mm, vias 2 -> 4
- net ROW5: track 501.7 -> 474.0 mm, vias 5 -> 4
- net GND: track 87.5 -> 113.7 mm, vias 2 -> 9
- net COL15: track 308.0 -> 330.9 mm, vias 1 -> 0
- net COL3: track 143.6 -> 165.7 mm
- net ROW3: track 377.2 -> 356.5 mm, vias 5 -> 4
- net COL16: track 328.1 -> 348.2 mm, vias 2 -> 0
- net COL13: track 237.2 -> 217.2 mm, vias 5 -> 1
- net ROW0: track 403.8 -> 386.4 mm, vias 3 -> 10
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
Commit message: cad
Parts:
- moved H7 327.7 mm to (21.7, 97.0)
- moved H3 251.0 mm to (63.5, 162.2)
- moved H1 177.0 mm to (376.4, 104.3)
- moved H5 116.1 mm to (264.8, 162.3)
